File: board/ESP32Eval/ESP32Eval.sch (KiCad schematic (older format))
At the start: 29 parts, among them J1 USB_B_Mini, J2 Conn_01x15, J3 Conn_01x15, Q1 Q_NPN_BCE, Q2 Q_NPN_BCE, SW1 SW_Flash, SW2 SW_Reset, U1 NCP1117-3.3_SOT223, U2 FT231XS, U3 ESP32-WROOM-32D

Commit message: Layout changes, added missing filter cap
Parts:
- removed Q1, Q2: Q_NPN_BCE, Package_TO_SOT_SMD:SOT-23_Handsoldering, symbol Device:Q_NPN_BCE
- added C10: 4,7µF, Capacitor_SMD:C_0805_2012Metric_Pad1.15x1.40mm_HandSolder, symbol Device:C
- added Q1, Q2: BC817, Package_TO_SOT_SMD:SOT-23, symbol Transistor_BJT:BC817
- C1, C4, C8: value C -> 10µF
- C2: value C -> 10nF
- C3, C5: value C -> 47pF
- C6, C7, C9: value C -> 100nF
- R1, R2: value R -> 27R
- R3, R6, R7: value R -> 270R
- R4, R5: value R -> 10k
Connections:
- net +5V: now also C10.1
- net GND: now also U2.7 (~DSR), U2.9 (~CTS), C10.2
- net at J2.4 (Pin_4), SW1.1, U3.25 (IO0): now also Q2.3 (C)
- net at J2.3 (Pin_3), SW2.1, U3.3 (EN): now also Q1.3 (C)
- net at R5.2, U2.1 (~DTR): now also Q2.2 (E)
- net at R4.2, U2.2 (~RTS): now also Q1.2 (E)
- net at R4.1: now also Q2.1 (B)
- net at R5.1: now also Q1.1 (B)
- no-connect marks 12 -> 11
Other:
- moved on the sheet: D2, D3, R6, R7
